File: pcb_v2.0-isolated-gate-control/pcb_v2.0-isolated-gate-control.kicad_sch (KiCad schematic)
At the start: 98 parts, among them J2 RS485, J3 LED 3,2V 20mA [-, +], J4 Fan [GND-supp, Diode, Mosfet], J5 2x Switch (to 5V), J6 Fan [GND/Mosfet-OUT, Diode, 2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, J7 Relay contacts [NO, COM, NC], J8 RS485, K2 24V relay, Q1 2N7000, Q2 2N7000, Q4 BC547, Q5 IRFZ24N, Q6 IRF3205, SW1 SW_SPDT, U1 MAX485E, U2 LM2576T-5, U3 ESP32_DevKit_V1_DOIT, U4 MAX485E

Commit message: pcb: outsrc isolated-dig-in, assign pins, Add supply, 12V out, servo-pwm
Parts:
- removed C10: 100n, Capacitor_THT:C_Disc_D7.0mm_W2.5mm_P5.00mm, symbol Device:C
- removed C2: 2200uf, Capacitor_THT:CP_Radial_D18.0mm_P7.50mm, symbol Device:C_Polarized
- removed D10, D11: D, Diode_THT:D_T-1_P12.70mm_Horizontal, symbol Device:D
- removed D14: TVS 1.5KE30A (starts 28.5V), Diode_THT:D_DO-201AE_P15.24mm_Horizontal, symbol Diode:PTVS5V0Z1USK
- removed F5: 500mA, Fuse:Fuseholder_Cylinder-5x20mm_Stelvio-Kontek_PTF78_Horizontal_Open, symbol Device:Fuse
- removed F6: (H7 24V 70W) -> 3A, Fuse:Fuseholder_Cylinder-5x20mm_Stelvio-Kontek_PTF78_Horizontal_Open, symbol Device:Fuse
- removed J6: Fan [GND/Mosfet-OUT, Diode, 24V-filtered], TerminalBlock:TerminalBlock_bornier-3_P5.08mm, symbol Connector:Screw_Terminal_01x03
- removed J7: Relay contacts [NO, COM, NC], TerminalBlock:TerminalBlock_bornier-3_P5.08mm, symbol Connector:Screw_Terminal_01x03
- removed K2: 24V relay, Relay_THT:Relay_SPDT_SANYOU_SRD_Series_Form_C, symbol Relay:SANYOU_SRD_Form_C
- removed OC1, OC2: LTV-817, Package_DIP:DIP-4_W10.16mm_LongPads, symbol Optocoupler_AKL:LTV-817
- removed Q6: IRF3205, Package_TO_SOT_THT:TO-220-3_Vertical, symbol Transistor_MOSFET_AKL:IRFZ24N
- removed R25, R28: 510, Resistor_THT:R_Axial_DIN0207_L6.3mm_D2.5mm_P10.16mm_Horizontal, symbol treiber-rescue:R
- removed R26, R27: 10k, Resistor_THT:R_Axial_DIN0207_L6.3mm_D2.5mm_P10.16mm_Horizontal, symbol Device:R
- removed R39: 10k, Resistor_THT:R_Axial_DIN0207_L6.3mm_D2.5mm_P10.16mm_Horizontal, symbol treiber-rescue:R
- removed R40, R41: 2k2, Resistor_THT:R_Axial_DIN0207_L6.3mm_D2.5mm_P10.16mm_Horizontal, symbol treiber-rescue:R
- removed SW1: SW_SPDT, symbol Switch:SW_SPDT
- added C10: 330nF, Capacitor_THT:C_Disc_D8.0mm_W5.0mm_P5.00mm, symbol treiber-rescue:C
- added C19: 100nF, Capacitor_THT:C_Disc_D7.0mm_W2.5mm_P5.00mm, symbol treiber-rescue:C
- added C20: 47u, Capacitor_THT:CP_Radial_D5.0mm_P2.50mm, symbol Device:C_Polarized
- added D22: D, Diode_THT:D_T-1_P12.70mm_Horizontal, symbol Device:D
- added F3: (H7 24V 70W) -> 3A, Fuse:Fuseholder_Cylinder-5x20mm_Stelvio-Kontek_PTF78_Horizontal_Open, symbol Device:Fuse
- added J1: ServoLock, TerminalBlock:TerminalBlock_bornier-3_P5.08mm, symbol Connector:Screw_Terminal_01x03
- added J10, J6: sw, TerminalBlock:TerminalBlock_bornier-2_P5.08mm, symbol Connector:Screw_Terminal_01x02
- added J11: sense, TerminalBlock:TerminalBlock_bornier-2_P5.08mm, symbol Connector:Screw_Terminal_01x02
- added J12: Relay contacts [NO, COM, NC], TerminalBlock:TerminalBlock_bornier-3_P5.08mm, symbol Connector:Screw_Terminal_01x03
- added J9: limit, symbol Connector:Screw_Terminal_01x04
- added K1: 24V relay, Relay_THT:Relay_SPDT_SANYOU_SRD_Series_Form_C, symbol Relay:SANYOU_SRD_Form_C
- added OC15, OC16, OC17, OC18, OC19, OC21: LTV-817, Package_DIP:DIP-4_W10.16mm_LongPads, symbol Optocoupler_AKL:LTV-817
- added R39, R41, R66, R68, R72, R77: 4k7, Resistor_THT:R_Axial_DIN0207_L6.3mm_D2.5mm_P10.16mm_Horizontal, symbol Device:R
- added R40, R65, R67, R71, R76: 330, Resistor_THT:R_Axial_DIN0207_L6.3mm_D2.5mm_P10.16mm_Horizontal, symbol Device:R
- added R64: 510, Resistor_THT:R_Axial_DIN0207_L6.3mm_D2.5mm_P10.16mm_Horizontal, symbol treiber-rescue:R
- added U5: L78S05CV_TO220, Package_TO_SOT_THT:TO-220-3_Vertical, symbol Regulator_Linear:LM7805_TO220
- added U6: ULN2803A, Package_DIP:DIP-18_W7.62mm_LongPads, symbol Transistor_Array:ULN2803A
- R10: value 2.5 -> 330; footprint Resistor_THT:R_Axial_DIN0922_L20.0mm_D9.0mm_P25.40mm_Horizontal -> Resistor_THT:R_Axial_DIN0207_L6.3mm_D2.5mm_P10.16mm_Horizontal
Connections:
- net +12V is gone; now on net +3V3: OC6.1
- net BUZZER is gone; now on net dOut_Buzzer: R13.2
- net LED is gone; now on net dOut_LED: R14.2
- net LED-ext is gone; now on net dOut_LED: R15.1
- net +24V filtered: now also D22.1 (K), K1.5; no longer C8.1, F2.2, PS1.2 (+VIN)
- net +3V3: now also OC16.1, OC17.1, OC18.1, OC19.1, OC21.1
- net +5VA: now also C19.1, C20.1, R39.1, R41.1, R66.1, R68.1, R72.1, R77.1, U5.3 (VO)
- net GND: now also C10.2, C19.2, C20.2, OC15.2, U5.2 (GND), U6.9 (GND); no longer OC6.3
- net GNDPWR: now also OC6.3, J1.3 (Pin_3), OC15.3, OC16.3, OC17.3, OC18.3, OC19.3, OC21.3
- net at F1.2: now also R11.1; no longer R10.1
- net at R10.2: now also OC6.2; no longer R11.1
- net at OC6.4: now also R39.2, U6.1 (I1)
- net dIn_Encoder2: now reaches U3.10 (GPIO27/ADC2)
- net dOut_EnLightBarriers: now reaches U3.11 (GPIO14/ADC2/HSPI_CLK)
- net dOut_EnLightBarriers: now also R71.1
- net dOut_RelayEnVFD2: now reaches U3.12 (GPIO12/HSPI-MISO/MTDI/[LOW-AT-BOOT])
- net dOut_RelayEnVFD2: now also R40.1
- net dOut_RelayEnVFD1: now reaches U3.13 (GPIO13/HSPI-MOSI)
- net dOut_RelayEnVFD1: now also R10.1
- net dOut_LED: now reaches U3.18 (GPIO15/HSPI_CS/MTDO/[HIGH-AT-BOOT])
- net dOut_LED: now also R67.1
- net dIn_RemoteOpen: now reaches U3.19 (GPIO2/ADC2)
- net dIn_Gate1-Open: now reaches U3.2 (GPIO36/ADC1-CH0/SENSOR_VP/[IN-ONLY])
- net dIn_LightBarrier: now reaches U3.23 (GPIO5/VSPI-CS)
- net dIn_Reserve: now reaches U3.24 (GPIO18/VSPI_CLK)
- net dOut_ServoPWM: now reaches U3.25 (GPIO19/VSPI-MISO)
- net dOut_ServoPWM: now also R76.1
- net dOut_Buzzer: now reaches U3.26 (GPIO21/I2C-SDA)
- net dOut_RelayEnServo: now reaches U3.29 (GPIO22/I2C-SCL)
- net dOut_RelayEnServo: now also R65.1
- net dIn_Gate1-Closed: now reaches U3.3 (GPIO39/ADC1-CH3/SENSOR_VN/[IN-ONLY])
- net dIn_Gate2-Open: now reaches U3.4 (GPIO34/ADC1-CH6//[IN-ONLY])
- net dIn_Gate2-Closed: now reaches U3.5 (GPIO35/ADC1-CH7/[IN-ONLY])
- net dIn_ButtonOpen: now reaches U3.6 (GPIO32/ADC1-CH4)
- net dIn_ButtonClose: now reaches U3.7 (GPIO33/ADC1-CH5)
- net dIn_RemoteClose: now reaches U3.8 (GPIO25/ADC2)
- net dIn_Encoder1: now reaches U3.9 (GPIO26/ADC2)
- new net: OC19.2, R71.2
- new net: OC19.4, R72.2, U6.5 (I5)
- new net: F3.1, K1.1
- new net: F3.2, J12.2 (Pin_2)
- new net: OC16.4, R41.2, U6.2 (I2)
- new net: D22.2 (A), K1.2, OC15.4
- new net: J12.3 (Pin_3), K1.3
- new net: J12.1 (Pin_1), K1.4
- new net: OC21.2, R76.2
- new net: J1.2 (Pin_2), OC21.4, R77.2
- new net: OC17.2, R65.2
- new net: OC17.4, R66.2, U6.3 (I3)
- new net: OC18.2, R67.2
- new net: OC18.4, R68.2, U6.4 (I4)
- new net: OC16.2, R40.2
- new net: OC15.1, R64.1
- new net +12V filtered: C10.1, C8.1, F2.2, PS1.2 (+VIN), U5.1 (VI), U6.10 (COM)
- new net dOut_RelayVFD1: R64.2
- new net isolated-digital-input_sw-to-gnd/in_switchToGND: J9.4 (Pin_4)
- new net isolated-digital-input_sw-to-gnd1/in_switchToGND: J9.3 (Pin_3)
- new net isolated-digital-input_sw-to-gnd2/in_switchToGND: J9.2 (Pin_2)
- new net isolated-digital-input_sw-to-gnd3/in_switchToGND: J9.1 (Pin_1)
- new net isolated-digital-input_sw-to-gnd4/in_switchToGND: J10.1 (Pin_1)
- new net isolated-digital-input_sw-to-gnd5/in_switchToGND: J10.2 (Pin_2)
- new net isolated-digital-input_sw-to-gnd6/in_switchToGND: J11.1 (Pin_1)
- new net isolated-digital-input_sw-to-gnd7/in_switchToGND: J11.2 (Pin_2)
- new net isolated-digital-input_sw-to-gnd8/in_switchToGND: J6.1 (Pin_1)
- new net isolated-digital-input_sw-to-gnd9/in_switchToGND: J6.2 (Pin_2)
Other:
- added sheet isolated-digital-input_sw-to-gnd (isolated-digital-input_sw-to-gnd.kicad_sch)
- added sheet isolated-digital-input_sw-to-gnd1 (isolated-digital-input_sw-to-gnd.kicad_sch)
- added sheet isolated-digital-input_sw-to-gnd10 (isolated-digital-input_sw-to-gnd.kicad_sch)
- added sheet isolated-digital-input_sw-to-gnd11 (isolated-digital-input_sw-to-gnd.kicad_sch)
- added sheet isolated-digital-input_sw-to-gnd2 (isolated-digital-input_sw-to-gnd.kicad_sch)
- added sheet isolated-digital-input_sw-to-gnd3 (isolated-digital-input_sw-to-gnd.kicad_sch)
- added sheet isolated-digital-input_sw-to-gnd4 (isolated-digital-input_sw-to-gnd.kicad_sch)
- added sheet isolated-digital-input_sw-to-gnd5 (isolated-digital-input_sw-to-gnd.kicad_sch)
- added sheet isolated-digital-input_sw-to-gnd6 (isolated-digital-input_sw-to-gnd.kicad_sch)
- added sheet isolated-digital-input_sw-to-gnd7 (isolated-digital-input_sw-to-gnd.kicad_sch)
- added sheet isolated-digital-input_sw-to-gnd8 (isolated-digital-input_sw-to-gnd.kicad_sch)
- added sheet isolated-digital-input_sw-to-gnd9 (isolated-digital-input_sw-to-gnd.kicad_sch)
- note added: "12V Supply (voltage filter)"
- note added: "5V Isolated Supply (dc-dc converter)"
- note added: "5V Supply (linear regulator)"
- note added: "Digital inputs (switch to GND, 12V pullup)"
- note added: "Driver 12V digital Outputs (Relays, led, servo-supply, barrier-supply)"
- note added: "PWM Signal out (Servo)"
- note added: "TODO: led connected to 12V outputs, buzzer directly to esp?"
- note added: "TODO: measure light barrier standby current, if high add circuit to enable only when closing"
- note added: "TODO: test if light barriers pull down when obstructed or free -> connect parallel or need and logic?"
- note removed: "24V Supply (voltage filter)"
- note removed: "5V Supply (isolated dc-dc converter)"
- note removed: "Digital input (switch to GND)"
- note removed: "Filter out 50V peaks on battery voltage each pwm cycle"
- note removed: "TODO: evaluate/test led current create sub-page for 6x reuse of this"
- note removed: "TVS: clamp to 12V short negative voltages"
- note removed: "low = fan on high = fan off"
- moved on the sheet: BZ1, C3, D6, F1, F2, J3, Q4, R13, R14, R15, R16

Commit message: pcb: Add Relays, mosfet-out, terminals, Fix RS485 isolation
Parts:
- removed C4: 100u, Capacitor_THT:CP_Radial_D8.0mm_P5.00mm, symbol Device:C_Polarized
- removed C5: 1000u, Capacitor_THT:CP_Radial_D10.0mm_P5.00mm, symbol Device:C_Polarized
- removed C6, C7: 100n, Capacitor_THT:C_Disc_D7.0mm_W2.5mm_P5.00mm, symbol Device:C
- removed D1: SM712_SOT23, Package_TO_SOT_SMD:SOT-23, symbol Diode:SM712_SOT23
- removed D4: 1N5822, Diode_THT:D_DO-201AD_P15.24mm_Horizontal, symbol Diode:1N5822
- removed D6: LED 3mm green 20mA 2.5V, LED_THT:LED_D3.0mm_Clear, symbol control-rescue:LED
- removed D7: D, Diode_THT:D_T-1_P12.70mm_Horizontal, symbol Device:D
- removed D8, D9: 5V1, Diode_THT:D_A-405_P10.16mm_Horizontal, symbol Device:D_Zener
- removed F2, F4: 500mA, Fuse:Fuseholder_Cylinder-5x20mm_Stelvio-Kontek_PTF78_Horizontal_Open, symbol Device:Fuse
- removed F3: (H7 24V 70W) -> 3A, Fuse:Fuseholder_Cylinder-5x20mm_Stelvio-Kontek_PTF78_Horizontal_Open, symbol Device:Fuse
- removed J12: Relay contacts [NO, COM, NC], TerminalBlock:TerminalBlock_bornier-3_P5.08mm, symbol Connector:Screw_Terminal_01x03
- removed J2: RS485, custom-footprints1:WAGO 733-363 Print-Stiftleiste, Micro, RM 2,5, gewinkelt, 3-pol, symbol Connector:Screw_Terminal_01x03
- removed J4: Fan [GND-supp, Diode, Mosfet], TerminalBlock:TerminalBlock_bornier-3_P5.08mm, symbol Connector:Screw_Terminal_01x03
- removed K1: 24V relay, Relay_THT:Relay_SPDT_SANYOU_SRD_Series_Form_C, symbol Relay:SANYOU_SRD_Form_C
- removed L1: 100u, Inductor_THT:L_Radial_D8.7mm_P5.00mm_Fastron_07HCP, symbol Device:L
- removed OC15: LTV-817, Package_DIP:DIP-4_W10.16mm_LongPads, symbol Optocoupler_AKL:LTV-817
- removed Q2: 2N7000, Package_TO_SOT_THT:TO-92_HandSolder, symbol Transistor_FET:2N7000
- removed Q4: BC547, Package_TO_SOT_THT:TO-92L, symbol Transistor_BJT_AKL:BC547
- removed Q5: IRFZ24N, Package_TO_SOT_THT:TO-220-3_Vertical, symbol Transistor_MOSFET_AKL:IRFZ24N
- removed R14: 130, Resistor_THT:R_Axial_DIN0207_L6.3mm_D2.5mm_P10.16mm_Horizontal, symbol control-rescue:R
- removed R15, R3: 470, Resistor_THT:R_Axial_DIN0207_L6.3mm_D2.5mm_P10.16mm_Horizontal, symbol Device:R
- removed R16: 100, Resistor_THT:R_Axial_DIN0207_L6.3mm_D2.5mm_P10.16mm_Horizontal, symbol Device:R
- removed R17: 1k, Resistor_THT:R_Axial_DIN0207_L6.3mm_D2.5mm_P10.16mm_Horizontal, symbol Device:R
- removed R18: 22k, Resistor_THT:R_Axial_DIN0207_L6.3mm_D2.5mm_P10.16mm_Horizontal, symbol Device:R
- removed R19, R20, R21, R22: 10k, Resistor_THT:R_Axial_DIN0207_L6.3mm_D2.5mm_P10.16mm_Horizontal, symbol control-rescue:R
- removed R2: 120, Resistor_THT:R_Axial_DIN0207_L6.3mm_D2.5mm_P2.54mm_Vertical, symbol Device:R
- removed R23, R24: 2k2, Resistor_THT:R_Axial_DIN0207_L6.3mm_D2.5mm_P10.16mm_Horizontal, symbol control-rescue:R
- removed R4, R9: 4k7, Resistor_THT:R_Axial_DIN0207_L6.3mm_D2.5mm_P10.16mm_Horizontal, symbol Device:R
- removed R5, R8: 200, Resistor_THT:R_Axial_DIN0207_L6.3mm_D2.5mm_P10.16mm_Horizontal, symbol Device:R
- removed R6: 6k2, Resistor_THT:R_Axial_DIN0207_L6.3mm_D2.5mm_P10.16mm_Horizontal, symbol Device:R
- removed R64: 510, Resistor_THT:R_Axial_DIN0207_L6.3mm_D2.5mm_P10.16mm_Horizontal, symbol treiber-rescue:R
- removed R7: 12k, Resistor_THT:R_Axial_DIN0207_L6.3mm_D2.5mm_P10.16mm_Horizontal, symbol Device:R
- removed TP1: TP UART RX, Connector_PinHeader_2.54mm:PinHeader_1x01_P2.54mm_Vertical, symbol Connector:TestPoint
- removed TP2: TP DIR, Connector_PinHeader_2.54mm:PinHeader_1x01_P2.54mm_Vertical, symbol Connector:TestPoint
- removed TP3: TP UART TX, Connector_PinHeader_2.54mm:PinHeader_1x01_P2.54mm_Vertical, symbol Connector:TestPoint
- removed U1: MAX485E, Package_SO:SOIC-8_3.9x4.9mm_P1.27mm, symbol Interface_UART:MAX485E
- removed U2: LM2576T-5, Package_TO_SOT_THT:TO-220-5_Vertical, symbol Regulator_Switching:LM2576T-5
- removed U3: ESP32_DevKit_V1_DOIT, ESP32_DevKit_V1_DOIT:esp32_devkit_v1_doit, symbol esp32_devkit_v1_doit:ESP32_DevKit_V1_DOIT
- added C4: 100n, Capacitor_THT:C_Disc_D7.0mm_W2.5mm_P5.00mm, symbol Device:C
- added D24: D, Diode_THT:D_T-1_P12.70mm_Horizontal, symbol Device:D
- added D26, D27: D, Diode_THT_AKL_Double:D_DO-27_P20.32mm_Horizontal, symbol Device:D
- added J12: Screw_Terminal_01x06, TerminalBlock_RND:TerminalBlock_RND_205-00016_1x06_P5.00mm_Horizontal, symbol Connector:Screw_Terminal_01x06
- added J13, J7: Relay contacts [NO, COM, NC], TerminalBlock:TerminalBlock_bornier-3_P5.08mm, symbol Connector:Screw_Terminal_01x03
- added J14, J2: sw, TerminalBlock:TerminalBlock_bornier-2_P5.08mm, symbol Connector:Screw_Terminal_01x02
- added J15, J16, J17, J18, J4: sense, TerminalBlock:TerminalBlock_bornier-2_P5.08mm, symbol Connector:Screw_Terminal_01x02
- added JP1, JP2, JP3: Jumper_2_Bridged, Jumper_AKL:Jumper_P2.54mm_D0.7mm, symbol Jumper:Jumper_2_Bridged
- added K1, K2: RT314A24, Relay_THT:Relay_SPDT_Schrack-RT1-16A-FormC_RM5mm, symbol Relay:RT314A24
- added OC23: LTV-817, Package_DIP:DIP-4_W10.16mm_LongPads, symbol Optocoupler_AKL:LTV-817
- added Q3, Q6: IRF5305, Package_TO_SOT_THT:TO-220-3_Vertical, symbol Transistor_MOSFET_AKL:IRF5305
- added R81: 330, Resistor_THT:R_Axial_DIN0207_L6.3mm_D2.5mm_P10.16mm_Horizontal, symbol Device:R
- added R82: 4k7, Resistor_THT:R_Axial_DIN0207_L6.3mm_D2.5mm_P10.16mm_Horizontal, symbol Device:R
- added R83, R84: 47k, Resistor_THT:R_Axial_DIN0207_L6.3mm_D2.5mm_P10.16mm_Horizontal, symbol Device:R
- added U1: esp32-devkit-v1_30Pin, devboards_libJonny:esp32-devkit-v1_30Pin, symbol relays_libJonny:esp32-devkit-v1_30Pin
- F1: footprint Fuse:Fuseholder_Cylinder-5x20mm_Stelvio-Kontek_PTF78_Horizontal_Open -> misc_libJonny:Fuseholder_Automotive-Regular_Fuse19x5x18mm_Footprint21x8mm_Inline
- J3: value LED 3,2V 20mA [-, +] -> sw
- J5: value 2x Switch (to 5V) -> sw
- J8: footprint custom-footprints1:WAGO 733-363 Print-Stiftleiste, Micro, RM 2,5, gewinkelt, 3-pol -> TerminalBlock:TerminalBlock_bornier-3_P5.08mm
- J9: footprint (none) -> TerminalBlock_Phoenix:TerminalBlock_Phoenix_MKDS-1,5-4_1x04_P5.00mm_Horizontal
- R1: value 470 -> 10k
- U4: footprint Package_SO:SOIC-8_3.9x4.9mm_P1.27mm -> Package_DIP_AKL:DIP-8_W7.62mm_LongPads
Connections:
- net +24V filtered is gone; now on net +12V filtered: D22.1 (K)
- net +12V filtered: now also C1.1, C3.1, D2.1 (K), D3.2 (A2), J3.1 (Pin_1), J3.2 (Pin_2), R11.2, R13.2, D24.1 (K), D26.2 (A), D27.2 (A), K1.A1, K2.A1, Q3.3 (S), Q6.3 (S), R83.2, R84.2
- net +3V3: now also J17.2 (Pin_2), OC23.1, U1.16 (3V3); no longer R1.1
- net +5V: now also J17.1 (Pin_1); no longer J3.1 (Pin_1)
- net +5VA: now also R29.1, U4.8 (VCC), C4.1, R82.1; no longer OC4.1
- net +BATT: now also J2.1 (Pin_1), J2.2 (Pin_2)
- net GND: now also J18.1 (Pin_1), J18.2 (Pin_2), U1.14 (GND), U1.17 (GND); no longer BZ1.2 (-), Q1.1 (S), U6.9 (GND)
- net GNDPWR: now also J5.1 (Pin_1), J5.2 (Pin_2), Q1.1 (S), U6.7 (I7), U6.8 (I8), U6.9 (GND), C4.2, J14.1 (Pin_1), J14.2 (Pin_2), J15.1 (Pin_1), J16.1 (Pin_1), OC23.3
- net RS485-UART_DIR-T: now also U1.20 (GPIO4/ADC2)
- net RS485-UART_TX: now also U1.22 (GPIO17/UART2-TX)
- net RS485_A: no longer R1.2
- net dIn_ButtonClose: now also U1.7 (GPIO33/ADC1-CH5)
- net dIn_ButtonOpen: now also U1.6 (GPIO32/ADC1-CH4)
- net dIn_Encoder1: now also U1.9 (GPIO26/ADC2)
- net dIn_Encoder2: now also U1.10 (GPIO27/ADC2)
- net dIn_Gate1-Closed: now also U1.3 (GPIO39/ADC1-CH3/SENSOR_VN/[IN-ONLY])
- net dIn_Gate1-Open: now also U1.2 (GPIO36/ADC1-CH0/SENSOR_VP/[IN-ONLY])
- net dIn_Gate2-Closed: now also U1.5 (GPIO35/ADC1-CH7/[IN-ONLY])
- net dIn_Gate2-Open: now also U1.4 (GPIO34/ADC1-CH6//[IN-ONLY])
- net dIn_LightBarrier: now also U1.23 (GPIO5/VSPI-CS)
- net dIn_RemoteClose: now also U1.8 (GPIO25/ADC2)
- net dIn_RemoteOpen: now also U1.19 (GPIO2/ADC2)
- net dIn_Reserve: now also U1.24 (GPIO18/VSPI_CLK)
- net dOut_Buzzer: now also R81.1, U1.26 (GPIO21/I2C-SDA); no longer R13.2
- net dOut_EnLightBarriers: now also U1.11 (GPIO14/ADC2/HSPI_CLK)
- net dOut_LED: now also U1.18 (GPIO15/HSPI_CS/MTDO/[HIGH-AT-BOOT])
- net dOut_RelayEnServo: now also U1.29 (GPIO22/I2C-SCL)
- net dOut_RelayEnVFD1: now also U1.13 (GPIO13/HSPI-MOSI)
- net dOut_RelayEnVFD2: now also U1.12 (GPIO12/HSPI-MISO/MTDI/[LOW-AT-BOOT])
- net dOut_ServoPWM: now also U1.25 (GPIO19/VSPI-MISO)
- net isolated-digital-input_sw-to-gnd10/in_switchToGND: now also J4.1 (Pin_1)
- net isolated-digital-input_sw-to-gnd11/in_switchToGND: now also J4.2 (Pin_2)
- net at D22.2 (A): now also JP2.2 (B), K1.A2
- net at D12.1 (K): now also U1.15 (VIN)
- net at Q1.2 (G): now also R1.1
- net at U4.1 (RO): now also R1.2; no longer R29.2
- net at Q1.3 (D): now also OC4.2
- net at U6.13 (O6): now also J12.6 (Pin_6), JP1.1 (A)
- net at U6.14 (O5): now also J12.5 (Pin_5), Q6.1 (G), R84.1
- net at U6.15 (O4): now also J12.4 (Pin_4)
- net at U6.16 (O3): now also J12.3 (Pin_3), Q3.1 (G), R83.1
- net at U6.17 (O2): now also J12.2 (Pin_2), JP2.1 (A)
- net at U6.18 (O1): now also J12.1 (Pin_1), JP3.1 (A)
- net at U6.6 (I6): now also OC23.4, R82.2
- net at C9.1: now also U1.1 (EN)
- net RS485-UART_RX renamed RS485-UART_RX_INVERTED
- net RS485-UART_RX_INVERTED: now also U1.21 (GPIO16/UART2-RX)
- new net: BZ1.2 (-), JP1.2 (B)
- new net: OC23.2, R81.2
- new net: J7.2 (Pin_2), K2.11
- new net: J7.1 (Pin_1), K2.12
- new net: J7.3 (Pin_3), K2.14
- new net: D24.2 (A), JP3.2 (B), K2.A2
- new net: D27.1 (K), J16.2 (Pin_2), Q6.2 (D)
- new net: J13.2 (Pin_2), K1.11
- new net: J13.1 (Pin_1), K1.12
- new net: J13.3 (Pin_3), K1.14
- new net: D26.1 (K), J15.2 (Pin_2), Q3.2 (D)
- new net: OC4.1, R29.2
Other:
- note added: "DIGITAL OUTPUTS - 5x open drain + 2x Relay, 2x high-side, Buzzer (VFD supply, Servo supply, LightBarrier supply, led, buzzer)"
- note added: "Isolated PWM Signal out (Servo)"
- note added: "Power terminals"
- note removed: "24V Relay: measured 16.7 mA at 30 V"
- note removed: "2x Digital input (Switches to 5V)"
- note removed: "3A overcurrent safe"
- note removed: "5V => 3.3V => R2/R1 = 1.941"
- note removed: "5V Supply (buck converter)"
- note removed: "7-40V"
- note removed: "Driver 12V digital Outputs (Relays, led, servo-supply, barrier-supply)"
- note removed: "From older projects, as reference"
- note removed: "Mosfet out (cooling Fan)"
- note removed: "Onboard Buzzer and LED"
- note removed: "PWM Signal out (Servo)"
- note removed: "Relay for Light"
- note removed: "TODO: add 5V linear regulator for MAX485"
- note removed: "TODO: led connected to 12V outputs, buzzer directly to esp?"
- note removed: "UART <-> RS485 non isolated, inverting"
- note removed: "external LED"
- moved on the sheet: C1, C10, C19, C20, C3, C8, C9, D12, D13, D2, D3, F1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

Commit message: pcb: Optinmize/protect PWM out, Start Layout (arrange as schematic)
Parts:
- added C5: 100uF, Capacitor_THT:CP_Radial_D18.0mm_P7.50mm, symbol Device:C_Polarized
- added D1: TVS 12V, Diode_THT:D_DO-41_SOD81_P12.70mm_Horizontal, symbol Diode:PTVS5V0Z1USK
- added F2: F-Servo, misc_libJonny:Fuseholder_Automotive-Regular_Fuse19x5x18mm_Footprint21x8mm_Inline, symbol Device:Fuse
- added Q2: 2N7000, Package_TO_SOT_THT:TO-92_HandSolder, symbol Transistor_FET:2N7000
- added R2: 200, Resistor_THT:R_Axial_DIN0207_L6.3mm_D2.5mm_P10.16mm_Horizontal, symbol Device:R
- added R3: 2k2, Resistor_THT:R_Axial_DIN0207_L6.3mm_D2.5mm_P10.16mm_Horizontal, symbol Device:R
- J10: value sw -> Buttons
- J11: value sense -> 2x encoder
- J13: value Relay contacts [NO, COM, NC] -> Relay VFD2 [NO, COM, NC]
- J14, J5: value sw -> GND-P
- J15: value sense -> Power-Servo-12V
- J16: value sense -> Power-LightBarrier-12V
- J17: value sense -> 3V3 5V VDD
- J18: value sense -> GNDD
- J2: value sw -> supply
- J3: value sw -> 12V-filtered
- J4: value sense -> light-barrier, reserve
- J6: value sw -> 2x remoteControl
- J7: value Relay contacts [NO, COM, NC] -> Relay VFD1 [NO, COM, NC]
Connections:
- net +3V3: no longer OC21.1
- net +5VA: now also R3.1
- net +BATT: now also F2.2
- net GND: now also OC21.2, C5.2
- net GNDPWR: now also D26.2 (A), D27.2 (A), J1.1 (Pin_1), D1.2 (A), Q2.1 (S); no longer J1.3 (Pin_3)
- net RS485_A: now also D13.2 (A2); no longer D13.1 (A1)
- net RS485_B: now also D13.1 (A1); no longer D13.2 (A2)
- net at D12.1 (K), U1.15 (VIN): now also C5.1
- net at R76.2: now also OC21.1; no longer OC21.2
- net at OC21.4, R77.2: now also Q2.2 (G); no longer J1.2 (Pin_2)
- net +12V filtered renamed +12V
- net +12V: no longer D26.2 (A), D27.2 (A)
- new net: D1.1 (K), Q2.3 (D), R2.1, R3.2
- new net: F2.1, J1.3 (Pin_3)
- new net: J1.2 (Pin_2), R2.2
Other:
- moved on the sheet: C10, C19, C20, C8, D26, D27, J1, J14, J17, J18, J2, J3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
