File: pcb_v2.0-isolated-gate-control/pcb_v2.0-isolated-gate-control.kicad_sch (KiCad schematic)
At the start: 96 parts, among them J1 ServoLock, J10 Buttons, J11 2x encoder, J12 limit-g2, J13 Relay VFD2 [NO, COM, NC], J14 GND-P, J15 OD, J16 Power-LightBarrier-12V, J17 3V3 5V VDD, J18 GNDD, J19 OD, J2 supply, J20 OD, J21 limit-g1, J3 12V-filtered, J4 light-barrier, reserve, J5 GND-P, J6 2x remoteControl, J7 Relay VFD1 [NO, COM, NC], J8 RS485, K1 RT314A24, K2 RT314A24, Q1 2N7000, Q2 2N7000, Q3 IRF5305, Q6 IRF5305, U1 esp32-devkit-v1_30Pin, U4 MAX485E, U5 L78S05CV_TO220, U6 ULN2803A

Commit message: pcb: remap gpio-pins, finish proof-of-concept routing (to evaluate arrangement)
Parts:
- C5: value 100uF -> 330uF; footprint Capacitor_THT:CP_Radial_D18.0mm_P7.50mm -> Capacitor_THT:CP_Radial_D10.0mm_P5.00mm
- R84: footprint Resistor_THT:R_Axial_DIN0207_L6.3mm_D2.5mm_P10.16mm_Horizontal -> Resistor_THT:R_Axial_DIN0207_L6.3mm_D2.5mm_P2.54mm_Vertical
Connections:
- net dIn_ButtonClose: now also U1.25 (GPIO19/VSPI-MISO); no longer U1.7 (GPIO33/ADC1-CH5)
- net dIn_ButtonOpen: now also U1.26 (GPIO21/I2C-SDA); no longer U1.6 (GPIO32/ADC1-CH4)
- net dIn_Encoder1: now also U1.5 (GPIO35/ADC1-CH7/[IN-ONLY]); no longer U1.9 (GPIO26/ADC2)
- net dIn_Encoder2: now also U1.6 (GPIO32/ADC1-CH4); no longer U1.10 (GPIO27/ADC2)
- net dIn_Gate1-Closed: now also U1.19 (GPIO2/ADC2); no longer U1.3 (GPIO39/ADC1-CH3/SENSOR_VN/[IN-ONLY])
- net dIn_Gate2-Closed: now also U1.24 (GPIO18/VSPI_CLK); no longer U1.5 (GPIO35/ADC1-CH7/[IN-ONLY])
- net dIn_Gate2-Open: now also U1.23 (GPIO5/VSPI-CS); no longer U1.4 (GPIO34/ADC1-CH6//[IN-ONLY])
- net dIn_LightBarrier: now also U1.3 (GPIO39/ADC1-CH3/SENSOR_VN/[IN-ONLY]); no longer U1.23 (GPIO5/VSPI-CS)
- net dIn_RemoteClose: now also U1.29 (GPIO22/I2C-SCL); no longer U1.8 (GPIO25/ADC2)
- net dIn_RemoteOpen: now also U1.30 (GPIO23/VSPI-MOSI); no longer U1.19 (GPIO2/ADC2)
- net dIn_Reserve: now also U1.4 (GPIO34/ADC1-CH6//[IN-ONLY]); no longer U1.24 (GPIO18/VSPI_CLK)
- net dOut_Buzzer: now also R67.1, U1.10 (GPIO27/ADC2); no longer R81.1, U1.26 (GPIO21/I2C-SDA)
- net dOut_EnLightBarriers: now also R65.1; no longer R71.1
- net dOut_LED: now also R10.1, U1.13 (GPIO13/HSPI-MOSI); no longer R67.1, U1.18 (GPIO15/HSPI_CS/MTDO/[HIGH-AT-BOOT])
- net dOut_RelayEnServo: now also R40.1, U1.12 (GPIO12/HSPI-MISO/MTDI/[LOW-AT-BOOT]); no longer R65.1, U1.29 (GPIO22/I2C-SCL)
- net dOut_RelayEnVFD1: now also R81.1, U1.8 (GPIO25/ADC2); no longer R10.1, U1.13 (GPIO13/HSPI-MOSI)
- net dOut_RelayEnVFD2: now also R71.1, U1.9 (GPIO26/ADC2); no longer R40.1, U1.12 (GPIO12/HSPI-MISO/MTDI/[LOW-AT-BOOT])
- net dOut_ServoPWM: now also U1.7 (GPIO33/ADC1-CH5); no longer U1.25 (GPIO19/VSPI-MISO)
Other:
- note added: "max out current: 200 mA max capactitive load: 1200 uF Short Circuit Protection: continuous, auto recovery"
- note removed: "Short Circuit Protection: continuous, auto recovery"
Changed lines of the file:
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@@
 	(wire
 		(pts
-			(xy 264.16 273.05) (xy 288.29 273.05)
-		)
-		(stroke
-			(width 0)
-			(type default)
-		)
-	)
-	(wire
-		(pts
 			(xy 85.09 82.55) (xy 105.41 82.55)
 		)
@@
 	(wire
 		(pts
-			(xy 195.58 242.57) (xy 213.36 242.57)
+			(xy 182.88 242.57) (xy 213.36 242.57)
 		)
 		(stroke
@@
 	(wire
 		(pts
-			(xy 281.94 245.11) (xy 304.8 245.11)
+			(xy 281.94 245.11) (xy 302.26 245.11)
 		)
 		(stroke
@@
 	(wire
 		(pts
-			(xy 288.29 273.05) (xy 288.29 250.19)
-		)
-		(stroke
-			(width 0)
-			(type default)
-		)
-	)
-	(wire
-		(pts
 			(xy 210.82 162.56) (xy 233.68 162.56)
 		)
@@
 	(wire
 		(pts
-			(xy 285.75 269.24) (xy 262.89 269.24)
-		)
-		(stroke
-			(width 0)
-			(type default)
-		)
-	)
-	(wire
-		(pts
 			(xy 63.5 34.29) (xy 74.93 34.29)
 		)
@@
 	(wire
 		(pts
-			(xy 195.58 245.11) (xy 213.36 245.11)
+			(xy 182.88 245.11) (xy 213.36 245.11)
 		)
 		(stroke
@@
 	(wire
 		(pts
+			(xy 281.94 247.65) (xy 299.72 247.65)
+		)
+		(stroke
+			(width 0)
+			(type default)
+		)
+	)
+	(wire
+		(pts
 			(xy 210.82 114.3) (xy 233.68 114.3)
 		)
@@
 	(wire
 		(pts
-			(xy 281.94 226.06) (xy 309.88 226.06)
+			(xy 281.94 226.06) (xy 300.99 226.06)
 		)
 		(stroke
@@
 	(wire
 		(pts
-			(xy 281.94 237.49) (xy 311.15 237.49)
+			(xy 281.94 237.49) (xy 316.23 237.49)
 		)
 		(stroke
@@
 	(wire
 		(pts
-			(xy 281.94 232.41) (xy 308.61 232.41)
+			(xy 281.94 232.41) (xy 316.23 232.41)
 		)
 		(stroke
@@
 	(wire
 		(pts
-			(xy 281.94 240.03) (xy 295.91 240.03)
+			(xy 281.94 240.03) (xy 302.26 240.03)
 		)
 		(stroke
@@
 	(wire
 		(pts
-			(xy 281.94 234.95) (xy 308.61 234.95)
+			(xy 281.94 234.95) (xy 316.23 234.95)
 		)
 		(stroke
@@
 	(wire
 		(pts
-			(xy 285.75 252.73) (xy 281.94 252.73)
+			(xy 281.94 252.73) (xy 300.99 252.73)
 		)
 		(stroke
@@
 	(wire
 		(pts
-			(xy 194.31 227.33) (xy 213.36 227.33)
+			(xy 193.04 227.33) (xy 213.36 227.33)
 		)
 		(stroke
@@
 	(wire
 		(pts
-			(xy 285.75 269.24) (xy 285.75 252.73)
-		)
-		(stroke
-			(width 0)
-			(type default)
-		)
-	)
-	(wire
-		(pts
 			(xy 30.48 276.86) (xy 53.34 276.86)
 		)
@@
 	(wire
 		(pts
-			(xy 195.58 247.65) (xy 213.36 247.65)
+			(xy 181.61 247.65) (xy 213.36 247.65)
 		)
 		(stroke
@@
 	(wire
 		(pts
-			(xy 194.31 229.87) (xy 213.36 229.87)
+			(xy 182.88 229.87) (xy 213.36 229.87)
 		)
 		(stroke
@@
 	(wire
 		(pts
-			(xy 281.94 223.52) (xy 298.45 223.52)
+			(xy 281.94 223.52) (xy 300.99 223.52)
 		)
 		(stroke
@@
 	(wire
 		(pts
-			(xy 281.94 250.19) (xy 288.29 250.19)
+			(xy 281.94 250.19) (xy 300.99 250.19)
 		)
 		(stroke
@@
 		)
 	)
-	(text "Short Circuit Protection: continuous, auto recovery"
+	(text "max out current: 200 mA\nmax capactitive load: 1200 uF\nShort Circuit Protection: continuous, auto recovery"
 		(exclude_from_sim no)
 		(at 175.006 53.848 0)
@@
 				(size 1.27 1.27)
 			)
+			(justify left)
 		)
 	)
@@
 	)
 	(label "dIn_Gate1-Closed"
-		(at 193.04 217.17 0)
+		(at 195.58 240.03 0)
 		(fields_autoplaced yes)
 		(effects
@@
 	)
 	(label "dIn_LightBarrier"
-		(at 262.89 269.24 0)
+		(at 193.04 217.17 0)
 		(fields_autoplaced yes)
 		(effects
@@
 	)
 	(label "dIn_Gate2-Closed"
-		(at 193.04 222.25 0)
+		(at 300.99 250.19 180)
 		(fields_autoplaced yes)
 		(effects
@@
 				(size 1.27 1.27)
 			)
-			(justify left bottom)
+			(justify right bottom)
 		)
 	)
@@
 	)
 	(label "dOut_EnLightBarriers"
-		(at 311.15 237.49 180)
+		(at 316.23 237.49 180)
 		(fields_autoplaced yes)
 		(effects
@@
 	)
 	(label "dOut_RelayEnServo"
-		(at 309.88 226.06 180)
+		(at 316.23 232.41 180)
 		(fields_autoplaced yes)
 		(effects
@@
 	)
 	(label "dIn_ButtonOpen"
-		(at 194.31 227.33 0)
+		(at 300.99 223.52 180)
 		(fields_autoplaced yes)
 		(effects
@@
 				(size 1.27 1.27)
 			)
-			(justify left bottom)
+			(justify right bottom)
 		)
 	)
@@
 	)
 	(label "dIn_Encoder1"
-		(at 195.58 245.11 0)
+		(at 193.04 222.25 0)
 		(fields_autoplaced yes)
 		(effects
@@
 	)
 	(label "dOut_Buzzer"
-		(at 298.45 223.52 180)
+		(at 182.88 247.65 0)
 		(fields_autoplaced yes)
 		(effects
@@
 				(size 1.524 1.524)
 			)
-			(justify right bottom)
+			(justify left bottom)
 		)
 	)
@@
 	)
 	(label "dIn_RemoteOpen"
-		(at 195.58 240.03 0)
+		(at 299.72 247.65 180)
 		(fields_autoplaced yes)
 		(effects
@@
 				(size 1.27 1.27)
 			)
-			(justify left bottom)
+			(justify right bottom)
 		)
 	)
 	(label "dOut_RelayEnServo"
-		(at 210.82 90.17 0)
+		(at 210.82 66.04 0)
 		(fields_autoplaced yes)
 		(effects
@@
 	)
 	(label "dOut_RelayEnVFD1"
-		(at 210.82 41.91 0)
+		(at 210.82 162.56 0)
 		(fields_autoplaced yes)
 		(effects
@@
 	)
 	(label "dOut_EnLightBarriers"
-		(at 210.82 138.43 0)
+		(at 210.82 90.17 0)
 		(fields_autoplaced yes)
 		(effects
@@
 	)
 	(label "dIn_ButtonClose"
-		(at 194.31 229.87 0)
+		(at 302.26 245.11 180)
 		(fields_autoplaced yes)
 		(effects
@@
 				(size 1.27 1.27)
 			)
-			(justify left bottom)
+			(justify right bottom)
 		)
 	)
@@
 	)
 	(label "dOut_ServoPWM"
-		(at 304.8 245.11 180)
+		(at 182.88 229.87 0)
 		(fields_autoplaced yes)
 		(effects
@@
 				(size 1.524 1.524)
 			)
-			(justify right bottom)
+			(justify left bottom)
 		)
 	)
 	(label "dOut_LED"
-		(at 210.82 114.3 0)
+		(at 210.82 41.91 0)
 		(fields_autoplaced yes)
 		(effects
@@
 	)
 	(label "dOut_LED"
-		(at 295.91 240.03 180)
+		(at 316.23 234.95 180)
 		(fields_autoplaced yes)
 		(effects
@@
 	)
 	(label "dOut_Buzzer"
-		(at 210.82 162.56 0)
+		(at 210.82 114.3 0)
 		(fields_autoplaced yes)
 		(effects
@@
 	)
 	(label "dIn_Gate2-Open"
-		(at 193.04 219.71 0)
+		(at 300.99 252.73 180)
 		(fields_autoplaced yes)
 		(effects
@@
 				(size 1.27 1.27)
 			)
-			(justify left bottom)
+			(justify right bottom)
 		)
 	)
@@
 	)
 	(label "dIn_Reserve"
-		(at 264.16 273.05 0)
+		(at 193.04 219.71 0)
 		(fields_autoplaced yes)
 		(effects
@@
 	)
 	(label "dOut_RelayEnVFD2"
-		(at 210.82 66.04 0)
+		(at 210.82 138.43 0)
 		(fields_autoplaced yes)
 		(effects
@@
 	)
 	(label "dIn_RemoteClose"
-		(at 195.58 242.57 0)
+		(at 300.99 226.06 180)
 		(fields_autoplaced yes)
 		(effects
@@
 				(size 1.27 1.27)
 			)
-			(justify left bottom)
+			(justify right bottom)
 		)
 	)
@@
 	)
 	(label "dOut_RelayEnVFD1"
-		(at 308.61 234.95 180)
+		(at 182.88 242.57 0)
 		(fields_autoplaced yes)
 		(effects
@@
 				(size 1.524 1.524)
 			)
-			(justify right bottom)
+			(justify left bottom)
 		)
 	)
 	(label "dOut_RelayEnVFD2"
-		(at 308.61 232.41 180)
+		(at 182.88 245.11 0)
 		(fields_autoplaced yes)
 		(effects
@@
 				(size 1.524 1.524)
 			)
-			(justify right bottom)
+			(justify left bottom)
 		)
 	)
@@
 	)
 	(label "dIn_Encoder2"
-		(at 195.58 247.65 0)
+		(at 193.04 227.33 0)
 		(fields_autoplaced yes)
 		(effects
@@
 			)
 		)
-		(property "Value" "100uF"
+		(property "Value" "330uF"
 			(at 222.25 187.0709 0)
 			(effects
@@
 			)
 		)
-		(property "Footprint" "Capacitor_THT:CP_Radial_D18.0mm_P7.50mm"
+		(property "Footprint" "Capacitor_THT:CP_Radial_D10.0mm_P5.00mm"
 			(at 225.0948 190.5 0)
 			(effects
@@
 			)
 		)
-		(property "Footprint" "Resistor_THT:R_Axial_DIN0207_L6.3mm_D2.5mm_P10.16mm_Horizontal"
+		(property "Footprint" "Resistor_THT:R_Axial_DIN0207_L6.3mm_D2.5mm_P2.54mm_Vertical"
 			(at 351.028 123.19 90)
 			(effects

Commit message: pcb: routing complete (DRC pass)
Connections:
- net +12V: no longer J3.2 (Pin_2)
- net +5VA: now also J3.2 (Pin_2)
Changed lines of the file:
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@@
 	)
 	(junction
-		(at 166.37 111.76)
-		(diameter 0)
-		(color 0 0 0 0)
-	)
-	(junction
 		(at 128.27 212.09)
 		(diameter 0)
@@
 	(wire
 		(pts
-			(xy 166.37 114.3) (xy 161.29 114.3)
+			(xy 161.29 114.3) (xy 171.45 114.3)
 		)
 		(stroke
@@
 	(wire
 		(pts
+			(xy 171.45 113.03) (xy 171.45 114.3)
+		)
+		(stroke
+			(width 0)
+			(type default)
+		)
+	)
+	(wire
+		(pts
 			(xy 193.04 227.33) (xy 213.36 227.33)
 		)
@@
 	(wire
 		(pts
-			(xy 166.37 111.76) (xy 166.37 114.3)
-		)
-		(stroke
-			(width 0)
-			(type default)
-		)
-	)
-	(wire
-		(pts
 			(xy 146.05 44.45) (xy 146.05 41.91)
 		)
@@
 					(unit 1)
 				)
+			)
+		)
+	)
+	(symbol
+		(lib_id "power:+5VA")
+		(at 171.45 113.03 0)
+		(unit 1)
+		(exclude_from_sim no)
+		(in_bom yes)
+		(on_board yes)
+		(dnp no)
+		(property "Reference" "#PWR029"
+			(at 171.45 116.84 0)
+			(effects
+				(font
+					(size 1.27 1.27)
+				)
+				(hide yes)
+			)
+		)
+		(property "Value" "+5VA"
+			(at 175.26 111.76 0)
+			(effects
+				(font
+					(size 1.27 1.27)
+				)
+			)
+		)
+		(property "Footprint" ""
+			(at 171.45 113.03 0)
+			(effects
+				(font
+					(size 1.27 1.27)
+				)
+				(hide yes)
+			)
+		)
+		(property "Datasheet" ""
+			(at 171.45 113.03 0)
+			(effects
+				(font
+					(size 1.27 1.27)
+				)
+				(hide yes)
+			)
+		)
+		(property "Description" "Power symbol creates a global label with name \"+5VA\""
+			(at 171.45 113.03 0)
+			(effects
+				(font
+					(size 1.27 1.27)
+				)
+				(hide yes)
+			)
+		)
+		(pin "1"
+		)
+		(instances
+			(project "pcb_v2.0-isolated-gate-control"
+				(path "/ac76819f-1531-4fd0-a2aa-e864e761b2bd"
+					(reference "#PWR029")
+					(unit 1)
+				)
