File: pcb_v2.0-isolated-gate-control/pcb_v2.0-isolated-gate-control.kicad_sch (KiCad schematic)
At the start: 96 parts, among them J1 ServoLock, J10 Buttons, J11 2x encoder, J12 limit-g2, J13 Relay VFD2 [NO, COM, NC], J14 GND-P, J15 OD, J16 Power-LightBarrier-12V, J17 3V3 5V VDD, J18 GNDD, J19 OD, J2 supply, J20 OD, J21 limit-g1, J3 12V-filtered, J4 light-barrier, reserve, J5 GND-P, J6 2x remoteControl, J7 Relay VFD1 [NO, COM, NC], J8 RS485, K1 RT314A24, K2 RT314A24, Q1 2N7000, Q2 2N7000, Q3 IRF5305, Q6 IRF5305, U1 esp32-devkit-v1_30Pin, U4 MAX485E, U5 L78S05CV_TO220, U6 ULN2803A

Commit message: pcb: Add text, testpoints, mounting-holes
Parts:
- removed U1: esp32-devkit-v1_30Pin, devboards_libJonny:esp32-devkit-v1_30Pin, symbol relays_libJonny:esp32-devkit-v1_30Pin
- added H1, H10, H11, H12, H13, H14, H2, H3, H4, H5, H6, H7, H8, H9: MountingHole_Pad, mountingHoles_libJonny:MountingHole_2.2mm_NPTH-with-pad_DRC-clearance-error, symbol Mechanical:MountingHole_Pad
- added J9: Conn_01x03_Pin, Connector_PinHeader_2.54mm:PinHeader_1x03_P2.54mm_Vertical, symbol Connector:Conn_01x03_Pin
- added TP1: TP DIR, Connector_PinHeader_2.54mm:PinHeader_1x01_P2.54mm_Vertical, symbol Connector:TestPoint
- added TP10: GND, Connector_PinHeader_2.54mm:PinHeader_1x01_P2.54mm_Vertical, symbol Connector:TestPoint
- added TP11, TP8: GNDPWR, Connector_PinHeader_2.54mm:PinHeader_1x01_P2.54mm_Vertical, symbol Connector:TestPoint
- added TP12: TP-servoPWM, Connector_PinHeader_2.54mm:PinHeader_1x01_P2.54mm_Vertical, symbol Connector:TestPoint
- added TP2: TP TX, Connector_PinHeader_2.54mm:PinHeader_1x01_P2.54mm_Vertical, symbol Connector:TestPoint
- added TP3: TP A, Connector_PinHeader_2.54mm:PinHeader_1x01_P2.54mm_Vertical, symbol Connector:TestPoint
- added TP5: TP B, Connector_PinHeader_2.54mm:PinHeader_1x01_P2.54mm_Vertical, symbol Connector:TestPoint
- added TP6: 12V, Connector_PinHeader_2.54mm:PinHeader_1x01_P2.54mm_Vertical, symbol Connector:TestPoint
- added TP7: 5V, Connector_PinHeader_2.54mm:PinHeader_1x01_P2.54mm_Vertical, symbol Connector:TestPoint
- added TP9: Vin, Connector_PinHeader_2.54mm:PinHeader_1x01_P2.54mm_Vertical, symbol Connector:TestPoint
- added U2: esp32-devkit-v1_30Pin, devboards_libJonny:esp32-devkit-v1_30Pin, symbol devboards_libJonny:esp32-devkit-v1_30Pin
- D1: value TVS 12V -> TVS 5V
- J3: value 12V-filtered -> 12V 5V
- TP4: value TP UART RX -> RX
Connections:
- net +12V: now also TP6.1
- net +3V3: now also J9.2 (Pin_2), U2.16 (3V3)
- net +5V: now also J9.3 (Pin_3)
- net +5VA: now also TP7.1
- net +BATT: now also TP9.1
- net GND: now also H1.1, H13.1, H14.1, H2.1, H3.1, J9.1 (Pin_1), TP10.1, U2.14 (GND), U2.17 (GND)
- net GNDPWR: now also H10.1, H11.1, H12.1, H4.1, H5.1, H6.1, H7.1, H8.1, H9.1, TP11.1, TP8.1
- net RS485-UART_DIR-T: now also TP1.1, U2.20 (GPIO4/ADC2)
- net RS485-UART_RX_INVERTED: now also U2.21 (GPIO16/UART2-RX)
- net RS485-UART_TX: now also TP2.1, U2.22 (GPIO17/UART2-TX)
- net RS485_A: now also TP3.1
- net RS485_B: now also TP5.1
- net Servo-PWM-Signal: now also TP12.1
- net dIn_ButtonClose: now also U2.25 (GPIO19/VSPI-MISO)
- net dIn_ButtonOpen: now also U2.26 (GPIO21/I2C-SDA)
- net dIn_Encoder1: now also U2.5 (GPIO35/ADC1-CH7/[IN-ONLY])
- net dIn_Encoder2: now also U2.6 (GPIO32/ADC1-CH4)
- net dIn_Gate1-Closed: now also U2.19 (GPIO2/ADC2)
- net dIn_Gate1-Open: now also U2.2 (GPIO36/ADC1-CH0/SENSOR_VP/[IN-ONLY])
- net dIn_Gate2-Closed: now also U2.24 (GPIO18/VSPI_CLK)
- net dIn_Gate2-Open: now also U2.23 (GPIO5/VSPI-CS)
- net dIn_LightBarrier: now also U2.3 (GPIO39/ADC1-CH3/SENSOR_VN/[IN-ONLY])
- net dIn_RemoteClose: now also U2.29 (GPIO22/I2C-SCL)
- net dIn_RemoteOpen: now also U2.30 (GPIO23/VSPI-MOSI)
- net dIn_Reserve: now also U2.4 (GPIO34/ADC1-CH6//[IN-ONLY])
- net dOut_Buzzer: now also U2.10 (GPIO27/ADC2)
- net dOut_EnLightBarriers: now also U2.11 (GPIO14/ADC2/HSPI_CLK)
- net dOut_LED: now also U2.13 (GPIO13/HSPI-MOSI)
- net dOut_RelayEnServo: now also U2.12 (GPIO12/HSPI-MISO/MTDI/[LOW-AT-BOOT])
- net dOut_RelayEnVFD1: now also U2.8 (GPIO25/ADC2)
- net dOut_RelayEnVFD2: now also U2.9 (GPIO26/ADC2)
- net dOut_ServoPWM: now also U2.7 (GPIO33/ADC1-CH5)
- net at C5.1, D12.1 (K): now also U2.15 (VIN)
- net at C9.1: now also U2.1 (EN)
Other:
- note added: "TODO: measure light barrier standby current, if high add circuit to enable only when closing TODO: test esp32 board with isolated supply + diode TODO: test digital input circuit (lowpass+optocoupler work?)"
- note added: "Testpoints power"
- note removed: "TODO: measure light barrier standby current, if high add circuit to enable only when closing"

Commit message: pcb: Add NOT-Gate (optocouplers off in idle), Replace ULN28 with 7Ch
Parts:
- removed U6: ULN2803A, Package_DIP:DIP-18_W7.62mm_LongPads, symbol Transistor_Array:ULN2803A
- added U1: ULN2003, Package_DIP:DIP-16_W7.62mm_LongPads, symbol Transistor_Array:ULN2003
- added U3: 74HC04, Package_DIP:DIP-14_W7.62mm_LongPads, symbol 74xx:74HC04
- R82: value 4k7 -> 10k
Connections:
- net +12V: now also U1.9 (COM)
- net +5VA: now also U3.14 (VCC)
- net GNDPWR: now also U1.7 (I7), U1.8 (GND), U3.7 (GND)
- net at J15.1 (Pin_1), JP1.1 (A): now also U1.13 (O4)
- net at OC19.4, R72.2: now also U3.11
- net at OC23.4, R82.2: now also U3.13
- net at OC16.4, R41.2: now also U3.3
- net at OC6.4, R39.2: now also U3.1
- net at OC17.4, R66.2: now also U3.5
- net at OC18.4, R68.2: now also U3.9
- net at J20.1 (Pin_1), JP3.1 (A): now also U1.11 (O6)
- net at J20.2 (Pin_2), JP2.1 (A): now also U1.12 (O5)
- net at J15.2 (Pin_2), Q6.1 (G), R84.1: now also U1.14 (O3)
- net at J19.1 (Pin_1), Q3.1 (G), R83.1: now also U1.15 (O2)
- net at J19.2 (Pin_2): now also U1.16 (O1)
- new net: U1.3 (I3), U3.6
- new net: U1.4 (I4), U3.8
- new net: U1.6 (I6), U3.12
- new net: U1.1 (I1), U3.2
- new net: U1.5 (I5), U3.10
- new net: U1.2 (I2), U3.4
Other:
- note added: "TODO: instead of ULN use USLN2003 (only 7 channel and available)"
- note added: "TODO: measure light barrier standby current, if high add circuit to enable only when closing test done: Photoelectric switch 12-24V NPN version https://www.aliexpress.com/item/1005001615723145.html - current when obstructed: 6mA - current when continous: <1mA (0.000A) - pulls low when obstructed - wires: brown=12V, blue=GND, black=collector TODO: test esp32 board with isolated supply + diode TODO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"
- note added: "invert the signal to - have low "off-state" current - prevent optocoupler led from being on in relay off-state - prevent optocoupler aging due to always on when outputs actually off"
- note removed: "TODO: measure light barrier standby current, if high add circuit to enable only when closing TODO: test esp32 board with isolated supply + diode TODO: test digital input circuit (lowpass+optocoupler work?)"
- moved on the sheet: BZ1, D22, D24, D26, D27, F2, J1, J13, J15, J16, J19, J20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

Commit message: pcb: Invert optocoupler-GPIO connection (high=output on), Layout adjusted (DRC pass)
Parts:
- J4: value light-barrier, reserve -> light-barrier, switch
- R39, R41, R66, R68, R72: value 4k7 -> 6k8
- R82: value 10k -> 6k8
Connections:
- net +3V3: no longer OC16.1, OC17.1, OC18.1, OC19.1, OC23.1, OC6.1
- net GND: now also OC16.2, OC17.2, OC18.2, OC19.2, OC23.2, OC6.2
- net at R71.2: now also OC19.1; no longer OC19.2
- net at R81.2: now also OC23.1; no longer OC23.2
- net at R10.2: now also OC6.1; no longer OC6.2
- net at R65.2: now also OC17.1; no longer OC17.2
- net at R67.2: now also OC18.1; no longer OC18.2
- net at R40.2: now also OC16.1; no longer OC16.2
- net dIn_Reserve renamed dIn_Switch
Other:
- note added: "- 5V IN (supply devboard) - 3V3 OUT (supply pullup resistors) - diode to prevent board from being supplied by usb cable (otherwise linear regulators get damaged when 9V not connected)"
- note added: "-[x] test if light barriers pull down when obstructed or free -> DONE: they pull to GND when obstructed -> no circuit necessary, connect both in parallel -[x] measure light barrier standby current, if high add circuit to enable only when closing -> DONE: Photoelectric switch 12-24V NPN version https://www.aliexpress.com/item/1005001615723145.html - current when obstructed: 6mA - current when cont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"
- note added: "Measurements with Optocoupler and 24V relay connected (15mA) 5 V, 200 Ohm -> I_led = 12 mA 5 V, 510 Ohm -> I_led = 7 mA, U_ce=0.7V 5 V, 820 Ohm -> I_led = 4.5 mA, U_ce=1.8V"
- note added: "Notes"
- note added: "Off/IDLE state: GPIO=low, optoLED=off, opto-out=high, ULN-in=low, ULN-out=floating, Relay=off / P-Mos-gate=high, P-Mos-out=floating => servo=off"
- note added: "TODO list"
- note added: "invert again using NOT-Gate so opto-led is OFF when outputs are OFF -> no 24/7 60mA current in "IDLE-state" -> prevent optocoupler from aging"
- note added: "supply NOT gate"
- note removed: "- 5V IN (supply devboard) - 3V3 OUT (supply i2c and levelshifter on board) - diode to prevent board from being supplied by usb cable (otherwise linear regulators get damaged when 9V not connected)"
- note removed: "Measurements with Optocoupler and 24V relay (15mA) 5 V, 200 Ohm -> I_led = 12 mA 5 V, 510 Ohm -> I_led = 7 mA, U_ce=0.7V 5 V, 820 Ohm -> I_led = 4.5 mA, U_ce=1.8V"
- note removed: "TODO: instead of ULN use USLN2003 (only 7 channel and available)"
- note removed: "TODO: measure light barrier standby current, if high add circuit to enable only when closing test done: Photoelectric switch 12-24V NPN version https://www.aliexpress.com/item/1005001615723145.html - current when obstructed: 6mA - current when continous: <1mA (0.000A) - pulls low when obstructed - wires: brown=12V, blue=GND, black=collector TODO: test esp32 board with isolated supply + diode TODO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"
- note removed: "TODO: test if light barriers pull down when obstructed or free -> connect parallel or need and logic?"
- note removed: "invert the signal to - have low "off-state" current - prevent optocoupler led from being on in relay off-state - prevent optocoupler aging due to always on when outputs actually off"
- moved on the sheet: BZ1, D22, D24, D26, D27, F2, J1, J13, J15, J16, J19, J20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

Commit message: pcb: Cleanup Schematic, arrange, replace legacy-symbols, optimize for ERC pass
Parts:
- #R13: symbol control-rescue:R -> Device:R
- C10, C19: symbol treiber-rescue:C -> Device:C
Connections:
- net RS485_A renamed RS485-A
- net RS485_B renamed RS485-B
- no-connect marks 0 -> 5
Other:
- note added: "HIGH in IDLE"
- note added: "INPUT"
- note added: "LOW in IDLE (receive)"
- note added: "MAX485 RO: ~1-3mA -> not enough for optocoupler led -> added MOS"
- note added: "Mountholes"
- note added: "RSO-2405S: - Input voltage range: 9V to 36V - max out current: 200 mA - max capactitive load: 1200 uF - Short Circuit Protection: continuous, auto recovery"
- note added: "TODO: when idling and not expecting to receive any data: deinitialize UART and turn DIR pin high in software. so DIR optocoupler led is off in idle"
- note added: "low when receiving"
- note added: "note: leds are controlled at cathode => non inverting signal ESP low -> led on -> MAX485 pulled low ESP high -> led off -> MAX485 high (pullup)"
- note removed: "Input voltage range: 9V to 36V"
- note removed: "MAX485 RO: ~1-3mA"
- note removed: "max out current: 200 mA max capactitive load: 1200 uF Short Circuit Protection: continuous, auto recovery"
- note removed: "note: leds are wired of inverted operation => non inverting signal ESP low -> led on -> MAX485 pulled low ESP high -> led off -> MAX485 high (pullup)"
- title: (none) -> pcb-isolated-gate-control
- moved on the sheet: C1, C10, C19, C20, C3, C4, D13, D2, D26, D3, F1, F2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

Commit message: pcb: finish todos, Fix esp32 power issues, document tests, dualType C footprint
Parts:
- added C6: 2200uF, Capacitor_THT:CP_Radial_D10.0mm_P5.00mm, symbol Device:C_Polarized
- C5: value 330uF -> 2200uF
- R31, R33: value 470 -> 330
Connections:
- net GND: now also C6.2
- net at C5.1, D12.1 (K), U2.15 (VIN): now also C6.1
Other:
- note added: "- 5V IN (supply devboard) - 3V3 OUT (supply pullup resistors) - diode to prevent backfeeding into the board by usb cable (dc-dc converter might get damaged)"
- note added: "Large buffer needed to compensate for 250 mA spikes at wifi startup (supply max 200 mA)"
- note removed: "- 5V IN (supply devboard) - 3V3 OUT (supply pullup resistors) - diode to prevent board from being supplied by usb cable (otherwise linear regulators get damaged when 9V not connected)"
- moved on the sheet: C5
Changed lines of the file:
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@@
 	)
 	(junction
+		(at 219.71 189.23)
+		(diameter 0)
+		(color 0 0 0 0)
+	)
+	(junction
 		(at 182.88 106.68)
 		(diameter 0)
@@
 	)
 	(junction
+		(at 226.06 179.07)
+		(diameter 0)
+		(color 0 0 0 0)
+	)
+	(junction
 		(at 191.77 146.05)
 		(diameter 0)
@@
 	(wire
 		(pts
-			(xy 231.14 181.61) (xy 231.14 190.5)
+			(xy 231.14 179.07) (xy 231.14 190.5)
 		)
 		(stroke
@@
 	(wire
 		(pts
+			(xy 219.71 189.23) (xy 226.06 189.23)
+		)
+		(stroke
+			(width 0)
+			(type default)
+		)
+	)
+	(wire
+		(pts
 			(xy 40.64 140.97) (xy 40.64 139.7)
 		)
@@
 	(wire
 		(pts
+			(xy 219.71 189.23) (xy 219.71 190.5)
+		)
+		(stroke
+			(width 0)
+			(type default)
+		)
+	)
+	(wire
+		(pts
 			(xy 40.64 151.13) (xy 39.37 151.13)
 		)
@@
 	(wire
 		(pts
+			(xy 226.06 187.96) (xy 226.06 189.23)
+		)
+		(stroke
+			(width 0)
+			(type default)
+		)
+	)
+	(wire
+		(pts
 			(xy 377.19 135.89) (xy 361.95 135.89)
 		)
@@
 	(wire
 		(pts
+			(xy 213.36 179.07) (xy 226.06 179.07)
+		)
+		(stroke
+			(width 0)
+			(type default)
+		)
+	)
+	(wire
+		(pts
 			(xy 334.01 187.96) (xy 334.01 189.23)
 		)
@@
 	(wire
 		(pts
+			(xy 213.36 179.07) (xy 213.36 180.34)
+		)
+		(stroke
+			(width 0)
+			(type default)
+		)
+	)
+	(wire
+		(pts
 			(xy 134.62 228.6) (xy 134.62 233.68)
 		)
@@
 	(wire
 		(pts
-			(xy 226.06 182.88) (xy 226.06 181.61)
-		)
-		(stroke
-			(width 0)
-			(type default)
-		)
-	)
-	(wire
-		(pts
 			(xy 384.81 101.6) (xy 382.27 101.6)
 		)
@@
 	(wire
 		(pts
+			(xy 213.36 189.23) (xy 213.36 187.96)
+		)
+		(stroke
+			(width 0)
+			(type default)
+		)
+	)
+	(wire
+		(pts
 			(xy 198.12 87.63) (xy 198.12 86.36)
 		)
@@
 	(wire
 		(pts
+			(xy 213.36 189.23) (xy 219.71 189.23)
+		)
+		(stroke
+			(width 0)
+			(type default)
+		)
+	)
+	(wire
+		(pts
 			(xy 179.07 146.05) (xy 182.88 146.05)
 		)
@@
 	(wire
 		(pts
-			(xy 226.06 181.61) (xy 231.14 181.61)
+			(xy 226.06 179.07) (xy 231.14 179.07)
 		)
 		(stroke
@@
 	(wire
 		(pts
+			(xy 226.06 180.34) (xy 226.06 179.07)
+		)
+		(stroke
+			(width 0)
+			(type default)
+		)
+	)
+	(wire
+		(pts
 			(xy 278.13 95.25) (xy 284.48 95.25)
 		)
@@
 	)
 	(rectangle
-		(start 317.246 206.248)
-		(end 406.654 250.444)
+		(start 317.246 201.168)
+		(end 406.654 251.714)
 		(stroke
 			(width 0)
@@
 		)
 	)
-	(text "\n  -[x] test if light barriers pull down when obstructed or free \n        -> DONE: they pull to GND when obstructed -> no circuit necessary, connect both in parallel\n\n  -[x] measure light barrier standby current, if high add circuit to enable only when closing\n	 -> DONE:\n	Photoelectric switch 12-24V NPN version https://www.aliexpress.com/item/1005001615723145.html\n		- current when obstructed: 6mA\n 		- current when continous: <1mA (0.000A)\n		- pulls low when obstructed\n		- wires: brown=12V, blue=GND, black=collector\n    -> circuit for cutting power added anyways\n\n  -[ ] test esp32 board with isolated supply + diode\n\n  -[ ] test digital input circuit (lowpass+optocoupler work?)\n\n  -[ ] 12V buzzer available? Footprint ok?\n\n  -[ ] test / evaluate optocoupler LED R with 3v3"
+	(text "\n  -[x] test if light barriers pull down when obstructed or free \n        -> DONE: they pull to GND when obstructed -> no circuit necessary, connect both in parallel\n\n  -[x] measure light barrier standby current, if high add circuit to enable only when closing\n	 -> DONE:\n	Photoelectric switch 12-24V NPN version https://www.aliexpress.com/item/1005001615723145.html\n		- current when obstructed: 6mA\n 		- current when continous: <1mA (0.000A)\n		- pulls low when obstructed\n		- wires: brown=12V, blue=GND, black=collector\n    -> circuit for cutting power added anyways\n\n  -[x] test esp32 board with isolated supply + diode\n	- when starting wifi at boot draws ~250 mA power insufficient -> boot loop\n    - when adden 2 x 2200 uF C after diode to buffer the peak it works reliably\n	- when running with wifi on draws ~125 mA continous\n    - => add additional C + prepare footprint for second DC DC converter inparallel?\n\n  -[x] test digital input circuit (lowpass+optocoupler work?)\n	- works well, lowpass turning off (open switch, pulls up to 12V) is faster than expected though \n	  due to RC charging up over led\n\n  -[x] test / evaluate optocoupler LED R with 3v3 => 330 Ohm -> 5 mA"
 		(exclude_from_sim no)
 		(at 316.23 229.362 0)
@@
 		)
 	)
+	(text "Large buffer needed to compensate for\n250 mA spikes at wifi startup\n(supply max 200 mA)"
+		(exclude_from_sim no)
+		(at 204.216 175.26 0)
+		(effects
+			(font
+				(size 1.2 1.2)
+			)
+			(justify left)
+		)
+	)
 	(text "1: used for USB\n3: used for USB"
 		(exclude_from_sim no)
@@
 		)
 	)
-	(text "- 5V IN (supply devboard)\n- 3V3 OUT (supply pullup resistors)\n- diode to prevent board from being supplied by usb cable\n  (otherwise linear regulators get damaged when 9V not connected)"
+	(text "- 5V IN (supply devboard)\n- 3V3 OUT (supply pullup resistors)\n- diode to prevent backfeeding into the board by usb cable\n  (dc-dc converter might get damaged)"
 		(exclude_from_sim no)
 		(at 256.032 181.356 0)
@@
 	(text "Fix boot issue while programming\nusing 10uF on enable pin"
 		(exclude_from_sim no)
-		(at 199.39 210.566 90)
+		(at 198.374 211.074 90)
 		(effects
 			(font
@@
 	(text "TODO list"
 		(exclude_from_sim no)
-		(at 327.406 210.058 0)
+		(at 326.644 204.978 0)
 		(effects
 			(font
@@
 			)
 		)
-		(property "Value" "470"
+		(property "Value" "330"
 			(at 52.578 270.764 90)
 			(effects
@@
 	)
 	(symbol
+		(lib_id "Device:C_Polarized")
+		(at 213.36 184.15 0)
+		(mirror y)
+		(unit 1)
+		(exclude_from_sim no)
+		(in_bom yes)
+		(on_board yes)
+		(dnp no)
+		(property "Reference" "C6"
+			(at 210.312 183.134 0)
+			(effects
+				(font
+					(size 1.27 1.27)
+				)
+				(justify left)
+			)
+		)
+		(property "Value" "2200uF"
+			(at 210.82 185.166 0)
+			(effects
+				(font
+					(size 1.27 1.27)
+				)
+				(justify left)
+			)
+		)
+		(property "Footprint" "Capacitor_THT:CP_Radial_D10.0mm_P5.00mm"
+			(at 212.3948 187.96 0)
+			(effects
+				(font
+					(size 1.27 1.27)
+				)
+				(hide yes)
+			)
+		)
+		(property "Datasheet" "~"
+			(at 213.36 184.15 0)
+			(effects
+				(font
+					(size 1.27 1.27)
+				)
+				(hide yes)
+			)
+		)
+		(property "Description" "Polarized capacitor"
+			(at 213.36 184.15 0)
+			(effects
+				(font
+					(size 1.27 1.27)
+				)
+				(hide yes)
+			)
+		)
+		(pin "2"
+		)
+		(pin "1"
+		)
+		(instances
+			(project "pcb_v2.0-isolated-gate-control"
+				(path "/ac76819f-1531-4fd0-a2aa-e864e761b2bd"
+					(reference "C6")
+					(unit 1)
+				)
+			)
+		)
+	)
+	(symbol
 		(lib_id "Optocoupler_AKL:LTV-817")
 		(at 152.4 156.21 0)
@@
 	(symbol
 		(lib_id "Device:C_Polarized")
-		(at 226.06 186.69 0)
+		(at 226.06 184.15 0)
 		(mirror y)
 		(unit 1)
@@
 		(dnp no)
 		(property "Reference" "C5"
-			(at 222.25 184.5309 0)
+			(at 223.012 183.388 0)
 			(effects
 				(font
@@
 			)
 		)
-		(property "Value" "330uF"
-			(at 222.25 187.0709 0)
+		(property "Value" "2200uF"
+			(at 223.52 185.166 0)
 			(effects
 				(font
@@
 		)
 		(property "Footprint" "Capacitor_THT:CP_Radial_D10.0mm_P5.00mm"
-			(at 225.0948 190.5 0)
+			(at 225.0948 187.96 0)
 			(effects
 				(font
@@
 		)
 		(property "Datasheet" "~"
-			(at 226.06 186.69 0)
+			(at 226.06 184.15 0)
 			(effects
 				(font
@@
 		)
 		(property "Description" "Polarized capacitor"
-			(at 226.06 186.69 0)
+			(at 226.06 184.15 0)
 			(effects
 				(font
@@
 	(symbol
 		(lib_id "power:GND")
-		(at 226.06 190.5 0)
+		(at 219.71 190.5 0)
 		(unit 1)
 		(exclude_from_sim no)
@@
 		(dnp no)
 		(property "Reference" "#PWR012"
-			(at 226.06 196.85 0)
+			(at 219.71 196.85 0)
 			(effects
 				(font
@@
 		)
 		(property "Value" "GND"
-			(at 222.504 190.754 0)
+			(at 216.154 192.278 0)
 			(effects
 				(font
@@
 		)
 		(property "Footprint" ""
-			(at 226.06 190.5 0)
+			(at 219.71 190.5 0)
 			(effects
 				(font
@@
 		)
 		(property "Datasheet" ""
-			(at 226.06 190.5 0)
+			(at 219.71 190.5 0)
 			(effects
 				(font
@@
 		)
 		(property "Description" "Power symbol creates a global label with name \"GND\" , ground"
-			(at 226.06 190.5 0)
+			(at 219.71 190.5 0)
 			(effects
 				(font
@@
 			)
 		)
-		(property "Value" "470"
+		(property "Value" "330"
 			(at 55.118 244.094 90)
 			(effects
