File: pcb_v2.0-isolated-gate-control/pcb_v2.0-isolated-gate-control.kicad_sch (KiCad schematic)
At the start: 124 parts, among them J1 ServoLock, J10 Buttons, J11 2x encoder, J12 limit-g2, J13 Relay VFD2 [NO, COM, NC], J14 GND-P, J15 OD, J16 Power-LightBarrier-12V, J17 3V3 5V VDD, J18 GNDD, J19 OD, J2 supply, J20 OD, J21 limit-g1, J3 12V 5V, J4 light-barrier, switch, J5 GND-P, J6 2x remoteControl, J7 Relay VFD1 [NO, COM, NC], J8 RS485, J9 Conn_01x03_Pin, K1 RT314A24, K2 RT314A24, Q1 2N7000, Q2 2N7000, Q3 IRF5305, Q6 IRF5305, U1 ULN2003, U2 esp32-devkit-v1_30Pin, U3 74HC04, U4 MAX485E, U5 L78S05CV_TO220

Commit message: pcb: Arrange silk/fab text, Mark front-solder, Add schematic+layout export
Parts:
- D3: value TVS 28V (starts 31V) -> TVS P6KE15A (12.8V)
Other:
- note added: "TODO"
- note removed: "TODO list"
Changed lines of the file:
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@@
 	(wire
 		(pts
-			(xy 306.07 80.01) (xy 306.07 78.74)
+			(xy 306.07 80.01) (xy 306.07 71.12)
 		)
 		(stroke
@@
 	(wire
 		(pts
-			(xy 304.8 80.01) (xy 306.07 80.01)
+			(xy 306.07 80.01) (xy 304.8 80.01)
 		)
 		(stroke
@@
 		)
 	)
-	(text "\n  -[x] test if light barriers pull down when obstructed or free \n        -> DONE: they pull to GND when obstructed -> no circuit necessary, connect both in parallel\n\n  -[x] measure light barrier standby current, if high add circuit to enable only when closing\n	 -> DONE:\n	Photoelectric switch 12-24V NPN version https://www.aliexpress.com/item/1005001615723145.html\n		- current when obstructed: 6mA\n 		- current when continous: <1mA (0.000A)\n		- pulls low when obstructed\n		- wires: brown=12V, blue=GND, black=collector\n    -> circuit for cutting power added anyways\n\n  -[x] test esp32 board with isolated supply + diode\n	- when starting wifi at boot draws ~250 mA power insufficient -> boot loop\n    - when adden 2 x 2200 uF C after diode to buffer the peak it works reliably\n	- when running with wifi on draws ~125 mA continous\n    - => add additional C + prepare footprint for second DC DC converter inparallel?\n\n  -[x] test digital input circuit (lowpass+optocoupler work?)\n	- works well, lowpass turning off (open switch, pulls up to 12V) is faster than expected though \n	  due to RC charging up over led\n\n  -[x] test / evaluate optocoupler LED R with 3v3 => 330 Ohm -> 5 mA"
+	(text "\n  -[x] test if light barriers pull down when obstructed or free \n        -> DONE: they pull to GND when obstructed -> no circuit necessary, connect both in parallel\n\n  -[x] measure light barrier standby current, if high add circuit to enable only when closing\n	 -> DONE:\n	Photoelectric switch 12-24V NPN version https://www.aliexpress.com/item/1005001615723145.html\n		- current when obstructed: 6mA\n 		- current when continous: <1mA (0.000A)\n		- pulls low when obstructed\n		- wires: brown=12V, blue=GND, black=collector\n    -> circuit for cutting power added anyways\n\n  -[x] test esp32 board with isolated supply + diode\n	- when starting wifi at boot draws ~250 mA power insufficient -> boot loop\n    - when adding 2 x 2200 uF C after diode to buffer the peak it works reliably\n	- when running with wifi on draws ~125 mA continous\n    - => add additional C (done) + prepare footprint for second DC DC converter in parallel?\n\n  -[x] test digital input circuit (lowpass+optocoupler work?)\n	- works well, lowpass turning off (open switch, pulls up to 12V) is faster than expected though \n	  due to RC charging up over led, see notes schematic sub-sheet\n\n  -[x] test / evaluate optocoupler LED R with 3v3 => 330 Ohm -> 5 mA"
 		(exclude_from_sim no)
 		(at 316.23 229.362 0)
@@
 		)
 	)
-	(text "TODO list"
+	(text "TODO"
 		(exclude_from_sim no)
-		(at 326.644 204.978 0)
+		(at 323.596 204.978 0)
 		(effects
 			(font
@@
 	(symbol
 		(lib_id "power:+24V")
-		(at 306.07 78.74 0)
+		(at 306.07 71.12 0)
 		(unit 1)
 		(exclude_from_sim no)
@@
 		(dnp no)
 		(property "Reference" "#PWR0131"
-			(at 306.07 82.55 0)
+			(at 306.07 74.93 0)
 			(effects
 				(font
@@
 		)
 		(property "Value" "+12V filtered"
-			(at 305.054 74.168 0)
+			(at 305.308 67.564 0)
 			(effects
 				(font
@@
 		)
 		(property "Footprint" ""
-			(at 306.07 78.74 0)
+			(at 306.07 71.12 0)
 			(effects
 				(font
@@
 		)
 		(property "Datasheet" ""
-			(at 306.07 78.74 0)
+			(at 306.07 71.12 0)
 			(effects
 				(font
@@
 		)
 		(property "Description" "Power symbol creates a global label with name \"+24V\""
-			(at 306.07 78.74 0)
+			(at 306.07 71.12 0)
 			(effects
 				(font
@@
 			)
 		)
-		(property "Value" "TVS 28V (starts 31V)"
-			(at 76.708 38.608 90)
+		(property "Value" "TVS P6KE15A (12.8V)"
+			(at 79.248 39.878 90)
 			(effects
 				(font

Commit message: pcb: Add Changelog, Note about GPIO-2 input issue
Connections:
- net dIn_Gate1-Closed: now also U2.24 (GPIO18/VSPI_CLK); no longer U2.19 (GPIO2/ADC2)
- net dIn_Gate1-Open: now also U2.23 (GPIO5/VSPI-CS); no longer U2.2 (GPIO36/ADC1-CH0/SENSOR_VP/[IN-ONLY])
- net dIn_Gate2-Closed: now also U2.19 (GPIO2/ADC2/[OnboardBlueLED+10k_down]); no longer U2.24 (GPIO18/VSPI_CLK)
- net dIn_Gate2-Open: now also U2.2 (GPIO36/ADC1-CH0/SENSOR_VP/[IN-ONLY]); no longer U2.23 (GPIO5/VSPI-CS)
Other:
- note added: "- Swap gpio assignment for limit-switches to match the engraved text - Add note about GPIO-2 (issues with using it as input)"
- note added: "-[ ] re-assign pins: use GPIO-2 as output instead of input due to onbard led and pulldown plus it has to be LOW when flashing"
- note added: "Changelog since Tag "pcb-for-V2-milled":"
- note added: "Note: Desolder blue LED + 10k pulldown R on DEVKITV1 so GPIO-2 works as intended as input. otherwise will be a voltage divider with the custom pullup -> 1.6V and always LOW remove module or "open gate" for flashing though since pin has to be LOW"
- note added: "TODO Next version:"
- note added: "TODO Pre-milling"
- note removed: "Measurements with Optocoupler and 24V relay connected (15mA) 5 V, 200 Ohm -> I_led = 12 mA 5 V, 510 Ohm -> I_led = 7 mA, U_ce=0.7V 5 V, 820 Ohm -> I_led = 4.5 mA, U_ce=1.8V"
- note removed: "Notes"
- note removed: "TODO"
- moved on the sheet: J9, TP10, TP11, TP6, TP7, TP8, TP9
