File: pcb_v2.0-isolated-gate-control/isolated-digital-input_sw-to-gnd.kicad_sch (KiCad schematic)
At the start: 7 parts

Commit message: pcb: Arrange silk/fab text, Mark front-solder, Add schematic+layout export
Parts:
- D23: value TVS 1.5KE30A (starts 28.5V) -> TVS P6KE15A (12.8V)
Other:
- note added: "Note: switch symbol only for illustrating the connection (nopop due to '#' in ref)"
- note added: "Notes made during testing this circuit: - Lowpass is extremely asymetric due to C additionally directly charging up over optocoupler led. -> better split R into two (one part between C and LED as well)? - R_filter = 3k3, C = 10uF: - 3.8ms delay turning on (switch closes to GND) - 0.1ms delay turning off (switch opens) - R = 2k2, C = 10uF - 2.5ms delay turning on - 0.5ms delay turning off - switch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"
- note added: "R value defined by 12V and optocoupler. Using required series R for led as R for lowpass at the same time. -> cant change value much to tune lowpass"
- note removed: "Note: switch symbol only for illustrating the connection (nopop due to #in ref)"
- note removed: "Notes made during testing this circuit: - Lowpass is extremely asymetric due to C additionally directly charging up over optocoupler led. -> better split R into two (one part between C and LED as well)? - R_filter = 3k3, C=10uF: - 3.8ms delay turning on (switch closes to GND) - 0.1ms delay turning off (switch opens) - R = 2k2, C = 10uF - 2.5ms delay turning on - 0.5ms delay turning off - switch b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"
- note removed: "R value defined by 12V and optocoupler. Using required series R for led as R for lowpass at the same time. -> cant change value much"
- moved on the sheet: D23
Changed lines of the file:
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@@
 	(wire
 		(pts
-			(xy 90.17 88.9) (xy 90.17 92.71)
+			(xy 90.17 85.09) (xy 90.17 92.71)
 		)
 		(stroke
@@
 	(wire
 		(pts
-			(xy 90.17 69.85) (xy 90.17 81.28)
+			(xy 90.17 69.85) (xy 90.17 77.47)
 		)
 		(stroke
@@
 		)
 	)
-	(text "Note: switch symbol only for \nillustrating the connection \n(nopop due to #in ref)"
+	(text "Note: switch symbol only for \nillustrating the connection \n(nopop due to '#' in ref)"
 		(exclude_from_sim no)
 		(at 41.402 57.912 0)
@@
 		)
 	)
-	(text "R value defined by 12V and optocoupler.\n Using required series R for led\n as R for lowpass at the same time.\n  -> cant change value much"
+	(text "R value defined by 12V and optocoupler.\n Using required series R for led\n as R for lowpass at the same time.\n  -> cant change value much to tune lowpass"
 		(exclude_from_sim no)
 		(at 101.6 28.702 0)
@@
 		)
 	)
-	(text "Notes made during testing this circuit:\n\n- Lowpass is extremely asymetric due to C additionally directly charging up over optocoupler led.\n	-> better split R into two (one part between C and LED as well)?\n\n- R_filter = 3k3,  C=10uF:\n	- 3.8ms delay turning on (switch closes to GND)\n	- 0.1ms delay turning off (switch opens)\n\n- R = 2k2, C = 10uF\n	- 2.5ms delay turning on\n	- 0.5ms delay turning off\n\n- switch bouncing is filtered well when using >= 1uF"
+	(text "Notes made during testing this circuit:\n\n- Lowpass is extremely asymetric due to C additionally directly charging up over optocoupler led.\n	-> better split R into two (one part between C and LED as well)?\n\n- R_filter = 3k3,  C = 10uF:\n	- 3.8ms delay turning on (switch closes to GND)\n	- 0.1ms delay turning off (switch opens)\n\n- R = 2k2, C = 10uF\n	- 2.5ms delay turning on\n	- 0.5ms delay turning off\n\n- switch bouncing is filtered well when using >= 1uF"
 		(exclude_from_sim no)
 		(at 37.338 117.094 0)
@@
 	(symbol
 		(lib_id "Diode:PTVS5V0Z1USK")
-		(at 90.17 85.09 270)
+		(at 90.17 81.28 270)
 		(unit 1)
 		(exclude_from_sim no)
@@
 		(dnp no)
 		(property "Reference" "D23"
-			(at 92.71 83.566 90)
+			(at 92.71 79.756 90)
 			(effects
 				(font
@@
 			)
 		)
-		(property "Value" "TVS 1.5KE30A (starts 28.5V)"
-			(at 60.452 85.598 90)
+		(property "Value" "TVS P6KE15A (12.8V)"
+			(at 67.31 81.534 90)
 			(effects
 				(font
@@
 		)
 		(property "Footprint" "Diode_THT:D_DO-41_SOD81_P12.70mm_Horizontal"
-			(at 85.725 85.09 0)
+			(at 85.725 81.28 0)
 			(effects
 				(font
@@
 		)
 		(property "Datasheet" "https://www.conrad.de/de/p/littelfuse-tvs-diode-1-5ke30a-do-201-28-5-v-1-5-kw-140796.html"
-			(at 90.17 85.09 0)
+			(at 90.17 81.28 0)
 			(effects
 				(font
@@
 		)
 		(property "Description" "5V, 1200W TVS unidirectional diode, DSN1608-2"
-			(at 90.17 85.09 0)
-			(effects
-				(font
+			(at 90.17 81.28 0)
+			(effects
+				(font
