File: pcb_v2.0-isolated-gate-control/pcb_v2.0-isolated-gate-control.kicad_pcb (KiCad board)
At the start: 4 copper layers, 170 x 110 mm, 195 parts, among them J1 ServoLock, J10 Buttons, J11 2x encoder, J12 limit-g2, J13 Relay VFD2 [NO, COM, NC], J14 GND-P, J15 OD, J16 Power-LightBarrier-12V, J17 3V3 5V VDD, J18 GNDD, J19 OD, J2 supply, J20 OD, J21 limit-g1, J3 12V 5V, J4 light-barrier, switch, J5 GND-P, J6 2x remoteControl, J7 Relay VFD1 [NO, COM, NC], J8 RS485, J9 Conn_01x03_Pin, K1 RT314A24, K2 RT314A24, Q1 2N7000, Q2 2N7000, Q3 IRF5305, Q6 IRF5305, U1 ULN2003, U2 esp32-devkit-v1_30Pin, U3 74HC04, U4 MAX485E, U5 L78S05CV_TO220

Commit message: pcb: Add Changelog, Note about GPIO-2 input issue
Connections:
- OC10 pad 4: /dIn_Gate2-Closed -> /dIn_Gate1-Closed
- OC7 pad 4: /dIn_Gate1-Open -> /dIn_Gate2-Open
- OC8 pad 4: /dIn_Gate1-Closed -> /dIn_Gate2-Closed
- OC9 pad 4: /dIn_Gate2-Open -> /dIn_Gate1-Open
- R42 pad 1: /dIn_Gate1-Open -> /dIn_Gate2-Open
- R45 pad 1: /dIn_Gate1-Closed -> /dIn_Gate2-Closed
- R48 pad 1: /dIn_Gate2-Open -> /dIn_Gate1-Open
- R51 pad 1: /dIn_Gate2-Closed -> /dIn_Gate1-Closed
- U2 pad 19: /dIn_Gate1-Closed -> /dIn_Gate2-Closed
- U2 pad 2: /dIn_Gate1-Open -> /dIn_Gate2-Open
- U2 pad 23: /dIn_Gate2-Open -> /dIn_Gate1-Open
- U2 pad 24: /dIn_Gate2-Closed -> /dIn_Gate1-Closed
Routing:
- net /dIn_Gate2-Closed: track 54.5 -> 87.6 mm, vias 0 -> 2
- net /dIn_Gate1-Closed: track 87.6 -> 54.5 mm, vias 2 -> 0
- net /dIn_Gate2-Open: track 65.4 -> 48.2 mm
- net /dIn_Gate1-Open: track 48.2 -> 65.4 mm
Other:
- board text added: "Desolder Blue LED + 10k R on ESP32-DevKit-V1 so GPIO-2 works as intended (digital input)"
- board text added: "Note: Input C2 must be LOW when flashing! alternatively remove esp32-board from pcb"
